Commit message: test

File: simulator/cart_pole_v0.urdf (robot description, URDF)
Before this commit: robot cart_pole, 5 links, 4 joints
Links:
- removed link left_border
- removed link right_border
Joints:
- removed joint slide_bar_to_left_border
- removed joint slide_bar_to_right_border
- joint cart_to_pole: axis 0 1 0 -> 0 -1 0; origin xyz=0.0 0.04 0 -> xyz=0.0 -0.04 0
- joint slider_to_cart: limit lower=-0.205 upper=0.205 effort=1000.0 velocity=10 -> lower=-2.0 upper=2.0 effort=1000.0 velocity=10
